File: PCB/DWM1000adapter/DWM1000_rev2.sch (EAGLE design)
At the start: 10 parts, among them IC1 DWM1000

Commit message: knas
Parts:
- removed SV3: (no value), con-lsta:FE05-1
- removed U$1: MICRO-USB-RECEPTACLE47589-0001, con-molex-usb:MICRO-USB-RECEPTACLE47589-0001
- removed U$2: PRO-MINI-2, Arduino-clone:PRO-MINI-2
- added SV2: (no value), con-lsta:FE08-1
- C1: device eagle-ltspice:CC0504 -> eagle-ltspice:CC1206
Connections:
- removed net 5V: U$1.1
- removed net 5V_RETURN: U$1.5
- removed net N$3: U$1.GND1
- removed net PGND: SV3.1, U$2.GND4
- removed net PRESET: SV3.5, U$2.DTR
- removed net PRX: SV3.3, U$2.RX1-1
- removed net PTX: SV3.4, U$2.TX0-1
- removed net PVCC: SV3.2, U$2.VCC1
- net 3.3: now also SV2.8; no longer U$2.RAW
- net CLK: now also SV2.5; no longer U$2.D13
- net CS: now also SV2.2; no longer U$2.D10
- net GND: now also SV2.1; no longer U$2.GND, U$2.GND2
- net IRQ: now also SV2.6; no longer U$2.D2
- net MISO: now also SV2.4; no longer U$2.D12
- net MOSI: now also SV2.3; no longer U$2.D11
- net RST: now also SV2.7; no longer U$2.D9
