File: PCB/DWM1000adapter/DWM1000_rev3_1.5mmdrill.brd (EAGLE design)
At the start: 34 x 32.3 mm, 8 parts, among them IC1 DWM1000

Commit message: added some stuff
Parts:
- SV2: device con-lsta:FE08 -> pin8:FE08
Routing:
- net IRQ: track 47.0 -> 49.9 mm
- net MOSI: track 24.5 -> 27.0 mm
- net CLK: track 37.3 -> 39.5 mm
- net MISO: track 31.1 -> 33.2 mm
- net RST: track 31.5 -> 32.7 mm
- net CS: track 14.6 -> 15.4 mm
Other:
- board text removed: "RX"
- board text removed: "TX"
Changed lines of the file:
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@@
 <?xml version="1.0" encoding="utf-8"?>
 <!DOCTYPE eagle SYSTEM "eagle.dtd">
-<eagle version="8.6.3">
+<eagle version="8.6.0">
 <drawing>
 <settings>
@@
 <wire x1="35.461" y1="28.88" x2="7.445" y2="28.88" width="0" layer="20"/>
 <wire x1="7.445" y1="28.88" x2="4.445" y2="25.88" width="0" layer="20" curve="90"/>
-<text x="13.335" y="8.89" size="0.889" layer="37">TX</text>
-<text x="26.416" y="9.017" size="0.889" layer="37">RX</text>
-<text x="16.002" y="0" size="1.143" layer="48" rot="R315">IRQ</text>
-<text x="18.669" y="0" size="1.143" layer="48" rot="R315">CLK</text>
-<text x="21.336" y="0" size="1.143" layer="48" rot="R315">MISO</text>
-<text x="23.749" y="0" size="1.143" layer="48" rot="R315">MOSI</text>
-<text x="26.289" y="0" size="1.143" layer="48" rot="R315">CS</text>
-<text x="28.956" y="0.127" size="1.27" layer="48" rot="R315">GND</text>
+<text x="16.256" y="-0.381" size="1.143" layer="48" rot="R315">IRQ</text>
+<text x="18.923" y="-0.381" size="1.143" layer="48" rot="R315">CLK</text>
+<text x="21.59" y="-0.381" size="1.143" layer="48" rot="R315">MISO</text>
+<text x="24.003" y="-0.381" size="1.143" layer="48" rot="R315">MOSI</text>
+<text x="26.543" y="-0.381" size="1.143" layer="48" rot="R315">CS</text>
+<text x="29.21" y="-0.254" size="1.27" layer="48" rot="R315">GND</text>
 <text x="5.969" y="13.462" size="1.524" layer="48" rot="R90" align="center">UWB Adapter</text>
 <text x="36.068" y="13.589" size="1.524" layer="48" rot="R90" align="center">Mikael &amp; Filip</text>
-<text x="10.541" y="0" size="1.27" layer="48" rot="R315">3.3</text>
+<text x="10.795" y="-0.381" size="1.27" layer="48" rot="R315">3.3</text>
 <hole x="7.112" y="26.416" drill="3"/>
 <hole x="35.814" y="26.416" drill="3"/>
 <hole x="7.112" y="-0.762" drill="3"/>
 <hole x="35.814" y="-0.762" drill="3"/>
-<text x="13.208" y="0" size="1.143" layer="48" rot="R315">RST</text>
+<text x="13.462" y="-0.381" size="1.143" layer="48" rot="R315">RST</text>
 </plain>
 <attributes>
@@
 <elements>
 <element name="IC1" library="decawave" package="DWM1000" value="DWM1000" x="20.32" y="27.051"/>
-<element name="SV2" library="con-lsta" library_urn="urn:adsk.eagle:library:161" package="FE08" package3d_urn="urn:adsk.eagle:package:8194/1" value="" x="19.939" y="6.731" rot="R180">
+<element name="SV2" library="pin8" package="FE08" value="" x="19.939" y="6.731" rot="R180">
 <attribute name="MF" value="" x="19.939" y="6.731" size="1.778" layer="27" rot="R180" display="off"/>
 <attribute name="MPN" value="" x="19.939" y="6.731" size="1.778" layer="27" rot="R180" display="off"/>
@@
 <contactref element="IC1" pad="3"/>
 <contactref element="SV2" pad="7"/>
-<wire x1="13.589" y1="6.731" x2="13.589" y2="4.699" width="0.4064" layer="1"/>
-<wire x1="13.589" y1="4.699" x2="13.081" y2="4.191" width="0.4064" layer="1"/>
-<wire x1="13.081" y1="4.191" x2="9.906" y2="4.191" width="0.4064" layer="1"/>
-<wire x1="9.906" y1="4.191" x2="8.001" y2="6.096" width="0.4064" layer="1"/>
-<wire x1="8.001" y1="6.096" x2="8.001" y2="14.097" width="0.4064" layer="1"/>
-<wire x1="8.001" y1="14.097" x2="7.747" y2="14.351" width="0.4064" layer="1"/>
-<wire x1="7.747" y1="14.351" x2="7.747" y2="18.034" width="0.4064" layer="1"/>
+<wire x1="7.747" y1="14.097" x2="7.747" y2="18.034" width="0.4064" layer="1"/>
 <wire x1="11.43" y1="21.717" x2="11.43" y2="24.511" width="0.4064" layer="1"/>
 <wire x1="11.43" y1="24.511" x2="11.97" y2="25.051" width="0.4064" layer="1"/>
 <wire x1="11.97" y1="25.051" x2="14.07" y2="25.051" width="0.4064" layer="1"/>
 <wire x1="7.747" y1="18.034" x2="11.43" y2="21.717" width="0.4064" layer="1"/>
+<wire x1="13.589" y1="6.731" x2="13.589" y2="4.191" width="0.4572" layer="1"/>
+<wire x1="13.589" y1="4.191" x2="12.954" y2="3.556" width="0.4572" layer="1"/>
+<wire x1="12.954" y1="3.556" x2="10.16" y2="3.556" width="0.4572" layer="1"/>
+<wire x1="10.16" y1="3.556" x2="7.747" y2="5.715" width="0.4572" layer="1"/>
+<wire x1="7.747" y1="5.715" x2="7.747" y2="14.097" width="0.4572" layer="1"/>
 </signal>
 <signal name="SPIPHA">
@@
 <wire x1="30.48" y1="25.4" x2="30.546" y2="25.019" width="0.5" layer="1"/>
 <wire x1="26.67" y1="25.4" x2="26.57" y2="25.051" width="0.5" layer="1"/>
-<wire x1="21.463" y1="1.524" x2="16.129" y2="6.731" width="0.5" layer="1"/>
-<wire x1="30.226" y1="1.524" x2="21.463" y2="1.524" width="0.5" layer="1"/>
-<wire x1="33.528" y1="4.699" x2="30.226" y2="1.524" width="0.5" layer="1"/>
-<wire x1="33.655" y1="21.59" x2="33.528" y2="4.699" width="0.5" layer="1"/>
-<wire x1="30.48" y1="24.765" x2="33.655" y2="21.59" width="0.5" layer="1"/>
+<wire x1="33.655" y1="21.59" x2="30.48" y2="24.765" width="0.5" layer="1"/>
 <wire x1="30.48" y1="24.765" x2="30.546" y2="25.019" width="0.5" layer="1"/>
+<wire x1="16.129" y1="6.731" x2="16.129" y2="5.207" width="0.4572" layer="1"/>
+<wire x1="16.129" y1="5.207" x2="20.447" y2="0.889" width="0.4572" layer="1"/>
+<wire x1="20.447" y1="0.889" x2="31.242" y2="0.889" width="0.4572" layer="1"/>
+<wire x1="31.242" y1="0.889" x2="34.163" y2="3.81" width="0.4572" layer="1"/>
+<wire x1="34.163" y1="3.81" x2="34.163" y2="21.209" width="0.4572" layer="1"/>
+<wire x1="34.163" y1="21.209" x2="34.036" y2="21.209" width="0.4572" layer="1"/>
+<wire x1="34.036" y1="21.209" x2="33.655" y2="21.59" width="0.4572" layer="1"/>
 </signal>
 <signal name="CLK">
@@
 <wire x1="27.94" y1="22.225" x2="26.67" y2="22.225" width="0.5" layer="1"/>
 <wire x1="32.639" y1="17.526" x2="27.94" y2="22.225" width="0.5" layer="1"/>
-<wire x1="32.512" y1="5.08" x2="32.639" y2="17.526" width="0.5" layer="1"/>
-<wire x1="29.845" y1="2.413" x2="32.512" y2="5.08" width="0.5" layer="1"/>
-<wire x1="22.733" y1="2.413" x2="29.845" y2="2.413" width="0.5" layer="1"/>
-<wire x1="18.669" y1="6.731" x2="22.733" y2="2.413" width="0.5" layer="1"/>
 <wire x1="26.67" y1="22.225" x2="26.57" y2="22.251" width="0.5" layer="1"/>
+<wire x1="18.669" y1="6.731" x2="18.669" y2="5.461" width="0.4572" layer="1"/>
+<wire x1="18.669" y1="5.461" x2="22.352" y2="1.778" width="0.4572" layer="1"/>
+<wire x1="22.352" y1="1.778" x2="30.48" y2="1.778" width="0.4572" layer="1"/>
+<wire x1="32.893" y1="17.272" x2="32.639" y2="17.526" width="0.4572" layer="1"/>
+<wire x1="30.48" y1="1.778" x2="32.893" y2="4.191" width="0.4572" layer="1"/>
+<wire x1="32.893" y1="4.191" x2="32.893" y2="17.272" width="0.4572" layer="1"/>
 </signal>
 <signal name="MISO">
@@
 <wire x1="27.94" y1="20.955" x2="26.67" y2="20.955" width="0.5" layer="1"/>
 <wire x1="31.496" y1="17.272" x2="27.94" y2="20.955" width="0.5" layer="1"/>
-<wire x1="31.496" y1="5.334" x2="31.496" y2="17.272" width="0.5" layer="1"/>
-<wire x1="29.464" y1="3.302" x2="31.496" y2="5.334" width="0.5" layer="1"/>
-<wire x1="24.257" y1="3.302" x2="29.464" y2="3.302" width="0.5" layer="1"/>
-<wire x1="21.209" y1="6.731" x2="24.257" y2="3.302" width="0.5" layer="1"/>
 <wire x1="26.67" y1="20.955" x2="26.57" y2="20.851" width="0.5" layer="1"/>
+<wire x1="21.209" y1="6.731" x2="21.209" y2="5.207" width="0.4572" layer="1"/>
+<wire x1="21.209" y1="5.207" x2="23.622" y2="2.794" width="0.4572" layer="1"/>
+<wire x1="23.622" y1="2.794" x2="29.972" y2="2.794" width="0.4572" layer="1"/>
+<wire x1="29.972" y1="2.794" x2="31.877" y2="4.699" width="0.4572" layer="1"/>
+<wire x1="31.877" y1="4.699" x2="31.877" y2="16.891" width="0.4572" layer="1"/>
+<wire x1="31.877" y1="16.891" x2="31.496" y2="17.272" width="0.4572" layer="1"/>
 </signal>
 <signal name="MOSI">
@@
 <wire x1="29.845" y1="12.7" x2="29.845" y2="17.145" width="0.5" layer="1"/>
 <wire x1="30.48" y1="12.065" x2="29.845" y2="12.7" width="0.5" layer="1"/>
-<wire x1="30.48" y1="5.715" x2="30.48" y2="12.065" width="0.5" layer="1"/>
-<wire x1="29.21" y1="4.445" x2="30.48" y2="5.715" width="0.5" layer="1"/>
-<wire x1="25.4" y1="4.445" x2="29.21" y2="4.445" width="0.5" layer="1"/>
-<wire x1="23.749" y1="6.731" x2="25.4" y2="4.445" width="0.5" layer="1"/>
 <wire x1="26.67" y1="19.05" x2="26.57" y2="19.451" width="0.5" layer="1"/>
+<wire x1="23.749" y1="6.731" x2="23.749" y2="4.191" width="0.4572" layer="1"/>
+<wire x1="23.749" y1="4.191" x2="24.003" y2="3.937" width="0.4572" layer="1"/>
+<wire x1="24.003" y1="3.937" x2="29.718" y2="3.937" width="0.4572" layer="1"/>
+<wire x1="29.718" y1="3.937" x2="30.734" y2="4.953" width="0.4572" layer="1"/>
+<wire x1="30.734" y1="4.953" x2="30.734" y2="11.811" width="0.4572" layer="1"/>
+<wire x1="30.734" y1="11.811" x2="30.48" y2="12.065" width="0.4572" layer="1"/>
 </signal>
 <signal name="CS">
@@
 <wire x1="24.13" y1="13.335" x2="25.4" y2="13.335" width="0.5" layer="1"/>
 <wire x1="23.495" y1="12.7" x2="24.13" y2="13.335" width="0.5" layer="1"/>
-<wire x1="23.495" y1="9.525" x2="23.495" y2="12.7" width="0.5" layer="1"/>
-<wire x1="26.289" y1="6.731" x2="23.495" y2="9.525" width="0.5" layer="1"/>
 <wire x1="26.67" y1="17.78" x2="26.57" y2="18.051" width="0.5" layer="1"/>
+<wire x1="26.289" y1="6.731" x2="26.289" y2="8.89" width="0.4572" layer="1"/>
+<wire x1="25.654" y1="9.525" x2="24.13" y2="9.525" width="0.4572" layer="1"/>
+<wire x1="24.13" y1="9.525" x2="23.495" y2="10.16" width="0.4572" layer="1"/>
+<wire x1="23.495" y1="10.16" x2="23.495" y2="12.7" width="0.4572" layer="1"/>
+<wire x1="26.289" y1="8.89" x2="25.654" y2="9.525" width="0.4572" layer="1"/>
 </signal>
 <signal name="3.3">
