File: PCB/UWBarduino/DWM1000_2.brd (EAGLE design)
At the start: 33.1 x 76.3 mm, 11 parts, among them IC1 DWM1000

Commit message: knas
Parts:
- C1: device eagle-ltspice:C0504 -> eagle-ltspice:C1206
- moved R3 18.4 mm to (31.5, 25.7), turned to 90 degrees
- moved U$1 5.59 mm to (2.79, -37.7)
- moved C1 3.18 mm to (9.91, 17.8), turned to 270 degrees
- moved SV3 3.18 mm to (32.5, -36.1)
- moved U$3 3.09 mm to (18.2, -41.1), turned to 90 degrees
- moved U$2 1.08 mm to (19.1, -15.5)
Connections:
- net GND: now also U$1.CASING1
- net N$3: now also U$1.CASING2; no longer U$1.CASING1
Routing:
- net GND: track 117.6 -> 190.6 mm, vias 1 -> 2
- net 3.3: track 117.5 -> 80.8 mm
- net RST: track 66.5 -> 38.0 mm, vias 0 -> 1
- net 5V: track 0.00 -> 18.9 mm
- net SPIPOL: track 12.0 -> 0.00 mm
- net SPIPHA: track 8.94 -> 0.00 mm
- net SYNC: track 8.72 -> 0.00 mm
- net WAKE: track 7.79 -> 0.00 mm
- net EXT: track 7.33 -> 0.00 mm
- net CLK: track 45.8 -> 51.8 mm, vias 1 -> 0
- net PGND: track 8.70 -> 14.0 mm
- net MISO: track 42.1 -> 46.6 mm, vias 0 -> 1
- net MOSI: track 34.1 -> 37.8 mm, vias 1 -> 0
- net PRX: track 15.9 -> 17.1 mm
- net CS: track 32.6 -> 33.3 mm
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- added copper zone on layer 1, net GND
- removed copper zone on layer 1, net N$4
Other:
- board size 33.1 x 76.3 mm -> 38.5 x 77.9 mm
- board text added: "GND"
- board text added: "Mikael & Filip"
- board text added: "Power in"
- board text added: "Prog in"
- board text added: "RST"
- board text added: "RX"
- board text added: "TX"
- board text added: "VCC"

Commit message: moa ros
Connections:
- net 5V: now also U$1.5; no longer U$1.1
- net GND: now also U$1.1; no longer U$1.5
Routing:
- net GND: track 190.6 -> 185.9 mm
- net 5V: track 18.9 -> 17.8 mm
Changed lines of the file:
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@@
 <layer number="14" name="Route14" color="1" fill="6" visible="no" active="no"/>
 <layer number="15" name="Route15" color="4" fill="6" visible="no" active="no"/>
-<layer number="16" name="Bottom" color="1" fill="1" visible="no" active="yes"/>
+<layer number="16" name="Bottom" color="1" fill="1" visible="yes" active="yes"/>
 <layer number="17" name="Pads" color="2" fill="1" visible="yes" active="yes"/>
 <layer number="18" name="Vias" color="2" fill="1" visible="yes" active="yes"/>
@@
 <wire x1="36.4818875" y1="28.626" x2="4.14789375" y2="28.626" width="0" layer="20"/>
 <wire x1="4.14789375" y1="28.626" x2="1.1479" y2="25.62033125" width="0" layer="20" curve="90.108265"/>
-<hole x="4.445" y="25.4" drill="3"/>
-<hole x="4.826" y="-45.974" drill="3"/>
-<hole x="35.941" y="-45.847" drill="3"/>
-<hole x="36.576" y="25.781" drill="3"/>
+<hole x="4.445" y="25.4" drill="2.2"/>
+<hole x="4.826" y="-45.974" drill="2.2"/>
+<hole x="35.941" y="-45.847" drill="2.2"/>
+<hole x="36.576" y="25.781" drill="2.2"/>
 <text x="3.556" y="-21.844" size="1.778" layer="48" rot="R270">Power in</text>
 <text x="32.639" y="-18.542" size="1.778" layer="48" rot="R270">Prog in</text>
@@
 <via x="9.779" y="24.892" extent="1-16" drill="1" diameter="1.778" shape="octagon"/>
 <wire x1="9.779" y1="24.892" x2="9.938" y2="25.051" width="0.508" layer="1"/>
-<wire x1="9.938" y1="25.051" x2="14.07" y2="25.051" width="0.508" layer="1"/>
+<wire x1="9.938" y1="25.051" x2="14.07" y2="25.051" width="0.5334" layer="1"/>
 </signal>
 <signal name="SPIPHA">
@@
 <contactref element="R3" pad="1"/>
 <contactref element="U$2" pad="D2"/>
-<wire x1="26.57" y1="25.051" x2="31.149" y2="25.051" width="0.508" layer="1"/>
+<wire x1="26.57" y1="25.051" x2="31.149" y2="25.051" width="0.5334" layer="1"/>
 <wire x1="31.149" y1="25.051" x2="31.496" y2="24.704" width="0.508" layer="1"/>
 <wire x1="31.496" y1="24.704" x2="35.306" y2="20.894" width="0.508" layer="1"/>
-<wire x1="35.306" y1="-10.668" x2="27.94" y2="-18.034" width="0.508" layer="1"/>
+<wire x1="35.306" y1="-10.668" x2="27.94" y2="-18.034" width="0.5334" layer="1"/>
 <wire x1="35.306" y1="20.894" x2="35.306" y2="-10.668" width="0.508" layer="1"/>
 </signal>
@@
 <contactref element="U$2" pad="GND"/>
 <contactref element="U$3" pad="3"/>
-<contactref element="U$1" pad="5"/>
 <polygon width="0.1524" layer="16">
 <vertex x="42.926" y="30.099"/>
@@
 <wire x1="9.906" y1="16.38" x2="9.906" y2="8.702" width="0.508" layer="1"/>
 <wire x1="9.906" y1="8.702" x2="11.115" y2="7.493" width="0.508" layer="1"/>
-<wire x1="2.794" y1="-33.544" x2="10.684" y2="-25.654" width="0.6096" layer="16"/>
-<wire x1="10.684" y1="-25.654" x2="11.176" y2="-25.654" width="0.6096" layer="16"/>
+<wire x1="2.794" y1="-33.544" x2="10.303" y2="-25.273" width="0.6096" layer="16"/>
+<wire x1="10.303" y1="-25.273" x2="11.176" y2="-25.654" width="0.6096" layer="16"/>
 <wire x1="21.971" y1="-39.878" x2="19.05" y2="-36.957" width="0.6096" layer="16"/>
 <wire x1="19.05" y1="-36.957" x2="14.732" y2="-36.957" width="0.6096" layer="16"/>
-<wire x1="14.732" y1="-36.957" x2="10.684" y2="-32.909" width="0.6096" layer="16"/>
-<wire x1="10.684" y1="-32.909" x2="10.684" y2="-25.654" width="0.6096" layer="16"/>
-<wire x1="5.594" y1="-39.019" x2="9.682" y2="-39.019" width="0.4572" layer="1"/>
-<wire x1="23.622" y1="-47.244" x2="25.273" y2="-45.593" width="0.4572" layer="1"/>
-<wire x1="25.273" y1="-45.593" x2="25.273" y2="-40.894" width="0.4572" layer="1"/>
-<wire x1="25.273" y1="-40.894" x2="24.257" y2="-39.878" width="0.4572" layer="1"/>
-<wire x1="24.257" y1="-39.878" x2="21.971" y2="-39.878" width="0.4572" layer="1"/>
-<wire x1="9.682" y1="-39.019" x2="17.907" y2="-47.244" width="0.4572" layer="1"/>
-<wire x1="17.907" y1="-47.244" x2="23.622" y2="-47.244" width="0.4572" layer="1"/>
+<wire x1="14.732" y1="-36.957" x2="10.303" y2="-32.528" width="0.6096" layer="16"/>
+<wire x1="10.303" y1="-32.528" x2="10.303" y2="-25.273" width="0.6096" layer="16"/>
 <wire x1="26.57" y1="23.651" x2="28.8" y2="23.651" width="0.7112" layer="1"/>
 <wire x1="30.81" y1="21.641" x2="31.144" y2="21.641" width="0.7112" layer="1"/>
 <wire x1="28.8" y1="23.651" x2="30.81" y2="21.641" width="0.7112" layer="1"/>
 <wire x1="26.57" y1="26.451" x2="26.57" y2="27.851" width="0.7112" layer="1"/>
+<contactref element="U$1" pad="1"/>
+<wire x1="5.594" y1="-36.419" x2="6.888" y2="-36.419" width="0.4064" layer="1"/>
+<wire x1="6.888" y1="-36.419" x2="7.874" y2="-35.433" width="0.4064" layer="1"/>
+<wire x1="7.874" y1="-35.433" x2="7.874" y2="-34.544" width="0.4064" layer="1"/>
+<wire x1="7.874" y1="-34.544" x2="7.874" y2="-33.401" width="0.4064" layer="1"/>
+<wire x1="7.874" y1="-33.401" x2="8.001" y2="-33.274" width="0.4064" layer="1"/>
+<wire x1="8.001" y1="-33.274" x2="4.0442125" y2="-33.274" width="0.4064" layer="1"/>
+<wire x1="4.0442125" y1="-33.274" x2="3.9110125" y2="-33.1408" width="0.4064" layer="1"/>
+<wire x1="3.9110125" y1="-33.1408" x2="2.794" y2="-33.1408" width="0.4064" layer="1"/>
+<wire x1="7.874" y1="-34.544" x2="10.16" y2="-36.83" width="0.4064" layer="1"/>
+<wire x1="10.16" y1="-36.83" x2="12.7" y2="-36.83" width="0.4064" layer="1"/>
+<wire x1="12.7" y1="-36.83" x2="15.748" y2="-39.878" width="0.4064" layer="1"/>
+<wire x1="15.748" y1="-39.878" x2="21.971" y2="-39.878" width="0.4064" layer="1"/>
 </signal>
 <signal name="N$1">
@@
 </signal>
 <signal name="5V">
-<contactref element="U$1" pad="1"/>
 <contactref element="U$3" pad="2"/>
-<wire x1="5.594" y1="-36.419" x2="9.114" y2="-36.419" width="0.4572" layer="1"/>
-<wire x1="15.113" y1="-42.418" x2="21.971" y2="-42.418" width="0.4572" layer="1"/>
-<wire x1="9.114" y1="-36.419" x2="15.113" y2="-42.418" width="0.4572" layer="1"/>
+<contactref element="U$1" pad="5"/>
+<wire x1="5.594" y1="-39.019" x2="11.079" y2="-39.019" width="0.6096" layer="1"/>
+<wire x1="11.079" y1="-39.019" x2="14.478" y2="-42.418" width="0.6096" layer="1"/>
+<wire x1="14.478" y1="-42.418" x2="21.971" y2="-42.418" width="0.6096" layer="1"/>
 </signal>
 <signal name="PRESET">
@@
 <contactref element="U$2" pad="GND3"/>
 <contactref element="SV3" pad="1"/>
-<wire x1="24.13" y1="-30.734" x2="24.13" y2="-28.321" width="0.5" layer="16"/>
-<wire x1="24.13" y1="-28.321" x2="25.527" y2="-26.924" width="0.5" layer="16"/>
-<wire x1="25.527" y1="-26.924" x2="30.099" y2="-26.924" width="0.5" layer="16"/>
-<wire x1="30.099" y1="-26.924" x2="32.512" y2="-29.337" width="0.5" layer="16"/>
-<wire x1="32.512" y1="-29.337" x2="32.512" y2="-30.988" width="0.5" layer="16"/>
+<wire x1="24.13" y1="-30.734" x2="24.13" y2="-28.321" width="0.5334" layer="16"/>
+<wire x1="24.13" y1="-28.321" x2="25.527" y2="-26.924" width="0.5334" layer="16"/>
+<wire x1="25.527" y1="-26.924" x2="30.099" y2="-26.924" width="0.5334" layer="16"/>
+<wire x1="30.099" y1="-26.924" x2="32.512" y2="-29.337" width="0.5334" layer="16"/>
+<wire x1="32.512" y1="-29.337" x2="32.512" y2="-30.988" width="0.5334" layer="16"/>
 </signal>
 <signal name="N$3">
